File: hardware/mini-pill/mini-pill.kicad_pcb (KiCad board)
At the start: 2 copper layers, 45 x 15 mm, 31 parts, among them J1 USB, J2 IO, U1 STM32F103C8Tx, U2 AP131-33, Y1 8MHz

Commit message: Add schematic
Other:
- board text added: "2023-10-14"
- board text removed: "2023-10-12"
Changed lines of the file:
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@@
       (plot_on_all_layers_selection 0x0000000_00000000)
       (disableapertmacros false)
-      (usegerberextensions false)
-      (usegerberattributes true)
-      (usegerberadvancedattributes true)
-      (creategerberjobfile true)
+      (usegerberextensions true)
+      (usegerberattributes false)
+      (usegerberadvancedattributes false)
+      (creategerberjobfile false)
       (dashed_line_dash_ratio 12.000000)
       (dashed_line_gap_ratio 3.000000)
@@
       (psa4output false)
       (plotreference true)
-      (plotvalue true)
+      (plotvalue false)
       (plotinvisibletext false)
       (sketchpadsonfab false)
-      (subtractmaskfromsilk false)
+      (subtractmaskfromsilk true)
       (outputformat 1)
       (mirror false)
-      (drillshape 1)
+      (drillshape 0)
       (scaleselection 1)
-      (outputdirectory "")
+      (outputdirectory "mini-pill-gerbers")
     )
   )
@@
     (effects (font (size 1 1) (thickness 0.15)) (justify left bottom mirror))
   )
-  (gr_text "2023-10-12" (at 134.8 64.5) (layer "B.SilkS")
+  (gr_text "2023-10-14" (at 134.8 64.5) (layer "B.SilkS")
     (effects (font (size 1.5 1.5) (thickness 0.3) bold) (justify left bottom mirror))
   )
